File: Eagle/Heizstabsteuerung.sch (EAGLE design)
At the start: 17 parts, among them U1 ESP32-DEVKITC-32D, X1 JST-XH-03-PIN-ROUND-PAD, X2 JST-XH-03-PIN-ROUND-PAD, X3 JST-XH-03-PIN-ROUND-PAD, X4 Versorgung

Commit message: Update V2.02 übertragen
Parts:
- removed LS_POWER_SENSOR1: BOB-12009, BOB-12009:BOB-12009
- removed SENSOR_L1, SENSOR_L2, SENSOR_L3: (no value), jumper:JP4E
- removed X1, X2, X3: JST-XH-03-PIN-ROUND-PAD, Rembrandt Electronics - JST XH Connectors v1-0:JST-XH-03-PIN-ROUND-PAD
- removed X4: Versorgung, con-wago-500:W237-102
- added C1, C2, C3: 10µF, Heizstabsteuerung:CPOL-EUE2.5-5
- added CON1: (no value), Heizstabsteuerung:WAGO-500-2
- added CON2, CON3, CON4: JST-XH-03, Heizstabsteuerung:JST-XH-03
- added JP3: L1, jumper:JP1E
- added JP4: L2, jumper:JP1E
- added JP5: L3, jumper:JP1E
- added LED3: gelb, Heizstabsteuerung:LED3MM
- added R10: 220, Heizstabsteuerung:R_10MM0207/10
- added R3, R5, R6, R7, R8, R9: 10k, Heizstabsteuerung:R_10MM0207/10
- added SV2: (no value), Heizstabsteuerung:FE06-1
- added U$1: LOGO_RAUCHSCHWALBE, Heizstabsteuerung:LOGO_RAUCHSCHWALBE
- JP1: value Display -> Display 16x2
- LED1: value red -> rot; device led:LED3MM -> Heizstabsteuerung:LED3MM
- LED2: device led:LED3MM -> Heizstabsteuerung:LED3MM
- LS_SSR1: value BOB-12009 -> LEVELSHIFTER; device BOB-12009:BOB-12009 -> Heizstabsteuerung:LEVELSHIFTER
- R1, R4: device rcl:R-EU_0204/7 -> Heizstabsteuerung:R_10MM0207/10
- R2: value 220 -> 330; device rcl:R-EU_0204/7 -> Heizstabsteuerung:R_10MM0207/10
- SV1: device con-lsta:FE06-1 -> Heizstabsteuerung:FE06-1
- U1: value ESP32-DEVKITC-32D -> ESP32-DEV-KIT-V4; device ESP32-DEVKITC-32D:ESP32-DEVKITC-32D -> Heizstabsteuerung:ESP32-DEV-KIT-V4
Connections:
- removed net GND$2: JP1.1, LED1.C, LED2.C, LS_POWER_SENSOR1.GND, LS_SSR1.GND, SENSOR_L1.3, SENSOR_L2.3, SENSOR_L3.3, SV1.5, U1.GND1, U1.GND2, U1.GND3, X1-3.S, X2-3.S, X3-3.S, X4-1.KL
- removed net N$24: LS_POWER_SENSOR1.HV3, SENSOR_L3.4
- removed net N$25: LS_POWER_SENSOR1.HV2, SENSOR_L2.4
- removed net N$26: LS_POWER_SENSOR1.HV1, SENSOR_L1.4
- removed net VDD3$13: LS_POWER_SENSOR1.LV, LS_SSR1.LV, R4.1, U1.3V3, X1-1.S, X2-1.S, X3-1.S
- removed net VDD5$3: JP1.2, LS_POWER_SENSOR1.HV, LS_SSR1.HV, SENSOR_L1.1, SENSOR_L2.1, SENSOR_L3.1, SV1.6, U1.EXT_5V, X4-2.KL
- new net +3V3: CON2.1, CON3.1, CON4.1, LS_SSR1.LV, R4.1, U1.3V3
- new net +5V: CON1.1, JP1.2, LS_SSR1.HV, R3.1, R6.1, R8.1, SV1.6, SV2.2, SV2.4, SV2.6, U1.EXT_5V
- new net GND: C1.-, C2.-, C3.-, CON1.2, CON2.3, CON3.3, CON4.3, JP1.1, LED1.C, LED2.C, LED3.C, LS_SSR1.GND, R5.2, R7.2, R9.2, SV1.5, SV2.1, SV2.3, SV2.5, U1.GND1, U1.GND2, U1.GND3
- new net N$17: R10.1, U1.IO4
- new net N$2: C1.+, JP3.2, R3.2, R5.1
- new net N$27: C2.+, JP4.2, R6.2, R7.1
- new net N$28: C3.+, JP5.2, R8.2, R9.1
- new net N$3: LED3.A, R10.2
- net N$11: now also CON2.2, CON3.2, CON4.2; no longer X1-2.S, X2-2.S, X3-2.S
- net N$12: now also JP3.1; no longer LS_POWER_SENSOR1.LV1
- net N$18: now also SV1.4; no longer SV1.1
- net N$19: now also SV1.3; no longer SV1.2
- net N$20: now also SV1.2; no longer SV1.3
- net N$21: now also JP4.1; no longer LS_POWER_SENSOR1.LV2
- net N$22: now also JP5.1; no longer LS_POWER_SENSOR1.LV3
- net N$9: now also SV1.1; no longer SV1.4
Other:
- note added: "Audio-Stecker GND"
- note added: "K-Leitung"
- note added: "L-Leitung"
- moved on the sheet: JP1, LED1, LED2, LS_SSR1, R1, R2, R4, SV1, U1
